Commit message: update urdf

File: Rice_description/urdf/materials.xacro (robot description, xacro)
@@ -1,5 +1,5 @@
 <?xml version="1.0" ?>
 <robot name="Rice" xmlns:xacro="http://www.ros.org/wiki/xacro" >
-<material name="silver">
+<material name="Rice_silver">
   <color rgba="0.700 0.700 0.700 1.000"/>
 </material>
