Commit message: update urdf

File: src/Rice_description/urdf/Rice.xacro (robot description, xacro)
@@ -6,6 +6,6 @@
 <link name="base_link">
   <inertial>
-    <origin xyz="-0.015971670540010845 -0.01298708868979309 0.9132275557142866" rpy="0 0 0"/>
-    <mass value="111.5224807340382"/>
+    <origin xyz="0.38402832945911597 0.567977724226758 0.9197289790734344" rpy="0 0 0"/>
+    <mass value="111.52248073403698"/>
     <inertia ixx="19.278738" iyy="11.892444" izz="29.802061" ixy="0.058745" iyz="0.077376" ixz="0.004947"/>
   </inertial>
@@ -26,10 +26,10 @@
 <link name="leg_br_1">
   <inertial>
-    <origin xyz="0.020674959041296737 0.059489197285151396 -0.4296056612393746" rpy="0 0 0"/>
-    <mass value="19.428196282242922"/>
+    <origin xyz="0.02067495895251792 0.05948901031816567 -0.42960523779205095" rpy="0 0 0"/>
+    <mass value="19.428196282242897"/>
     <inertia ixx="0.69198" iyy="0.64895" izz="0.118365" ixy="-0.016967" iyz="-0.04479" ixz="-0.001759"/>
   </inertial>
   <visual>
-    <origin xyz="-0.37 0.555 -0.87" rpy="0 0 0"/>
+    <origin xyz="-0.77 -0.025965 -0.876501" rpy="0 0 0"/>
     <geometry>
       <mesh filename="file://$(find Rice_description)/meshes/leg_br_1.stl" scale="0.001 0.001 0.001"/>
@@ -38,5 +38,5 @@
   </visual>
   <collision>
-    <origin xyz="-0.37 0.555 -0.87" rpy="0 0 0"/>
+    <origin xyz="-0.77 -0.025965 -0.876501" rpy="0 0 0"/>
     <geometry>
       <mesh filename="file://$(find Rice_description)/meshes/leg_br_1.stl" scale="0.001 0.001 0.001"/>
@@ -46,10 +46,10 @@
 <link name="leg_bl_1">
   <inertial>
-    <origin xyz="-0.02020942421503935 0.05818411411251201 -0.4348060760754819" rpy="0 0 0"/>
-    <mass value="19.903337256280803"/>
+    <origin xyz="-0.020209424216131984 0.05818392702927147 -0.4348056527161479" rpy="0 0 0"/>
+    <mass value="19.9033372562808"/>
     <inertia ixx="0.720932" iyy="0.676639" izz="0.120784" ixy="0.017565" iyz="-0.050773" ixz="0.003917"/>
   </inertial>
   <visual>
-    <origin xyz="0.4 0.555 -0.87" rpy="0 0 0"/>
+    <origin xyz="-0.0 -0.025965 -0.876501" rpy="0 0 0"/>
     <geometry>
       <mesh filename="file://$(find Rice_description)/meshes/leg_bl_1.stl" scale="0.001 0.001 0.001"/>
@@ -58,5 +58,5 @@
   </visual>
   <collision>
-    <origin xyz="0.4 0.555 -0.87" rpy="0 0 0"/>
+    <origin xyz="-0.0 -0.025965 -0.876501" rpy="0 0 0"/>
     <geometry>
       <mesh filename="file://$(find Rice_description)/meshes/leg_bl_1.stl" scale="0.001 0.001 0.001"/>
@@ -66,10 +66,10 @@
 <link name="leg_fr_1">
   <inertial>
-    <origin xyz="0.020209424439251666 -0.05818411429774317 -0.43480607531996185" rpy="0 0 0"/>
-    <mass value="19.90333719348548"/>
+    <origin xyz="0.020209424438183965 -0.058184301381010606 -0.43480565196065807" rpy="0 0 0"/>
+    <mass value="19.90333719348541"/>
     <inertia ixx="0.720932" iyy="0.676639" izz="0.120784" ixy="0.017565" iyz="0.050773" ixz="-0.003917"/>
   </inertial>
   <visual>
-    <origin xyz="-0.37 -0.535 -0.87" rpy="0 0 0"/>
+    <origin xyz="-0.77 -1.115965 -0.876501" rpy="0 0 0"/>
     <geometry>
       <mesh filename="file://$(find Rice_description)/meshes/leg_fr_1.stl" scale="0.001 0.001 0.001"/>
@@ -78,5 +78,5 @@
   </visual>
   <collision>
-    <origin xyz="-0.37 -0.535 -0.87" rpy="0 0 0"/>
+    <origin xyz="-0.77 -1.115965 -0.876501" rpy="0 0 0"/>
     <geometry>
       <mesh filename="file://$(find Rice_description)/meshes/leg_fr_1.stl" scale="0.001 0.001 0.001"/>
@@ -86,10 +86,10 @@
 <link name="leg_fl_1">
   <inertial>
-    <origin xyz="-0.020233756049858553 -0.05820262908497592 -0.4347334415519548" rpy="0 0 0"/>
-    <mass value="19.897003188386847"/>
+    <origin xyz="-0.020233756052453953 -0.058202816166196714 -0.4347330181911013" rpy="0 0 0"/>
+    <mass value="19.897003188386865"/>
     <inertia ixx="0.72058" iyy="0.676271" izz="0.120724" ixy="-0.017537" iyz="0.050689" ixz="0.003807"/>
   </inertial>
   <visual>
-    <origin xyz="0.4 -0.535 -0.87" rpy="0 0 0"/>
+    <origin xyz="-0.0 -1.115965 -0.876501" rpy="0 0 0"/>
     <geometry>
       <mesh filename="file://$(find Rice_description)/meshes/leg_fl_1.stl" scale="0.001 0.001 0.001"/>
@@ -98,5 +98,5 @@
   </visual>
   <collision>
-    <origin xyz="0.4 -0.535 -0.87" rpy="0 0 0"/>
+    <origin xyz="-0.0 -1.115965 -0.876501" rpy="0 0 0"/>
     <geometry>
       <mesh filename="file://$(find Rice_description)/meshes/leg_fl_1.stl" scale="0.001 0.001 0.001"/>
@@ -106,70 +106,70 @@
 <link name="wheel_br_1">
   <inertial>
-    <origin xyz="-0.0036583592135003284 7.882583474838611e-15 -1.1379786002407855e-15" rpy="0 0 0"/>
-    <mass value="65.80472593736364"/>
+    <origin xyz="-0.0036583592134993292 -1.8708468446995696e-07 4.2335822600381157e-07" rpy="0 0 0"/>
+    <mass value="65.80472593736363"/>
+    <inertia ixx="1.584128" iyy="0.836383" izz="0.836383" ixy="0.0" iyz="0.0" ixz="-0.0"/>
+  </inertial>
+  <visual>
+    <origin xyz="-0.863 -0.025965 -0.206501" rpy="0 0 0"/>
+    <geometry>
+      <mesh filename="file://$(find Rice_description)/meshes/wheel_br_1.stl" scale="0.001 0.001 0.001"/>
+    </geometry>
+    <material name="silver"/>
+  </visual>
+  <collision>
+    <origin xyz="-0.863 -0.025965 -0.206501" rpy="0 0 0"/>
+    <geometry>
+      <mesh filename="file://$(find Rice_description)/meshes/wheel_br_1.stl" scale="0.001 0.001 0.001"/>
+    </geometry>
+  </collision>
+</link>
+<link name="wheel_fr_1">
+  <inertial>
+    <origin xyz="-0.0036583592134961096 -1.8708470195250015e-07 4.233582252821666e-07" rpy="0 0 0"/>
+    <mass value="65.80472593736363"/>
+    <inertia ixx="1.584128" iyy="0.836383" izz="0.836383" ixy="-0.0" iyz="0.0" ixz="0.0"/>
+  </inertial>
+  <visual>
+    <origin xyz="-0.863 -1.115965 -0.206501" rpy="0 0 0"/>
+    <geometry>
+      <mesh filename="file://$(find Rice_description)/meshes/wheel_fr_1.stl" scale="0.001 0.001 0.001"/>
+    </geometry>
+    <material name="silver"/>
+  </visual>
+  <collision>
+    <origin xyz="-0.863 -1.115965 -0.206501" rpy="0 0 0"/>
+    <geometry>
+      <mesh filename="file://$(find Rice_description)/meshes/wheel_fr_1.stl" scale="0.001 0.001 0.001"/>
+    </geometry>
+  </collision>
+</link>
+<link name="wheel_bl_1">
+  <inertial>
+    <origin xyz="0.0020000000000000573 -1.870846836303508e-07 4.233582258372781e-07" rpy="0 0 0"/>
+    <mass value="65.80472593736363"/>
+    <inertia ixx="1.584128" iyy="0.836383" izz="0.836383" ixy="-0.0" iyz="0.0" ixz="0.0"/>
+  </inertial>
+  <visual>
+    <origin xyz="0.093 -0.025965 -0.206501" rpy="0 0 0"/>
+    <geometry>
+      <mesh filename="file://$(find Rice_description)/meshes/wheel_bl_1.stl" scale="0.001 0.001 0.001"/>
+    </geometry>
+    <material name="silver"/>
+  </visual>
+  <collision>
+    <origin xyz="0.093 -0.025965 -0.206501" rpy="0 0 0"/>
+    <geometry>
+      <mesh filename="file://$(find Rice_description)/meshes/wheel_bl_1.stl" scale="0.001 0.001 0.001"/>
+    </geometry>
+  </collision>
+</link>
+<link name="wheel_fl_1">
+  <inertial>
+    <origin xyz="0.0020000000000037488 -1.8708469617934043e-07 4.2335822519889987e-07" rpy="0 0 0"/>
+    <mass value="65.80472593736363"/>
     <inertia ixx="1.584128" iyy="0.836383" izz="0.836383" ixy="0.0" iyz="0.0" ixz="0.0"/>
   </inertial>
   <visual>
-    <origin xyz="-0.463 0.555 -0.2" rpy="0 0 0"/>
-    <geometry>
-      <mesh filename="file://$(find Rice_description)/meshes/wheel_br_1.stl" scale="0.001 0.001 0.001"/>
-    </geometry>
-    <material name="silver"/>
-  </visual>
-  <collision>
-    <origin xyz="-0.463 0.555 -0.2" rpy="0 0 0"/>
-    <geometry>
-      <mesh filename="file://$(find Rice_description)/meshes/wheel_br_1.stl" scale="0.001 0.001 0.001"/>
-    </geometry>
-  </collision>
-</link>
-<link name="wheel_fr_1">
-  <inertial>
-    <origin xyz="-0.003658359213496276 -9.43689570931383e-15 -2.498001805406602e-16" rpy="0 0 0"/>
-    <mass value="65.80472593736364"/>
-    <inertia ixx="1.584128" iyy="0.836383" izz="0.836383" ixy="-0.0" iyz="-0.0" ixz="-0.0"/>
-  </inertial>
-  <visual>
-    <origin xyz="-0.463 -0.535 -0.2" rpy="0 0 0"/>
-    <geometry>
-      <mesh filename="file://$(find Rice_description)/meshes/wheel_fr_1.stl" scale="0.001 0.001 0.001"/>
-    </geometry>
-    <material name="silver"/>
-  </visual>
-  <collision>
-    <origin xyz="-0.463 -0.535 -0.2" rpy="0 0 0"/>
-    <geometry>
-      <mesh filename="file://$(find Rice_description)/meshes/wheel_fr_1.stl" scale="0.001 0.001 0.001"/>
-    </geometry>
-  </collision>
-</link>
-<link name="wheel_bl_1">
-  <inertial>
-    <origin xyz="0.0019999999999998352 7.882583474838611e-15 -1.9984014443252818e-15" rpy="0 0 0"/>
-    <mass value="65.80472593736363"/>
-    <inertia ixx="1.584128" iyy="0.836383" izz="0.836383" ixy="-0.0" iyz="0.0" ixz="0.0"/>
-  </inertial>
-  <visual>
-    <origin xyz="0.493 0.555 -0.2" rpy="0 0 0"/>
-    <geometry>
-      <mesh filename="file://$(find Rice_description)/meshes/wheel_bl_1.stl" scale="0.001 0.001 0.001"/>
-    </geometry>
-    <material name="silver"/>
-  </visual>
-  <collision>
-    <origin xyz="0.493 0.555 -0.2" rpy="0 0 0"/>
-    <geometry>
-      <mesh filename="file://$(find Rice_description)/meshes/wheel_bl_1.stl" scale="0.001 0.001 0.001"/>
-    </geometry>
-  </collision>
-</link>
-<link name="wheel_fl_1">
-  <inertial>
-    <origin xyz="0.002000000000003721 -3.774758283725532e-15 -5.828670879282072e-16" rpy="0 0 0"/>
-    <mass value="65.80472593736361"/>
-    <inertia ixx="1.584128" iyy="0.836383" izz="0.836383" ixy="0.0" iyz="0.0" ixz="-0.0"/>
-  </inertial>
-  <visual>
-    <origin xyz="0.493 -0.535 -0.2" rpy="0 0 0"/>
+    <origin xyz="0.093 -1.115965 -0.206501" rpy="0 0 0"/>
     <geometry>
       <mesh filename="file://$(find Rice_description)/meshes/wheel_fl_1.stl" scale="0.001 0.001 0.001"/>
@@ -178,5 +178,5 @@
   </visual>
   <collision>
-    <origin xyz="0.493 -0.535 -0.2" rpy="0 0 0"/>
+    <origin xyz="0.093 -1.115965 -0.206501" rpy="0 0 0"/>
     <geometry>
       <mesh filename="file://$(find Rice_description)/meshes/wheel_fl_1.stl" scale="0.001 0.001 0.001"/>
@@ -185,26 +185,26 @@
 </link>
 <joint name="Revolute 9" type="continuous">
-  <origin xyz="0.37 -0.555 0.87" rpy="0 0 0"/>
+  <origin xyz="0.77 0.025965 0.876501" rpy="0 0 0"/>
   <parent link="base_link"/>
   <child link="leg_br_1"/>
-  <axis xyz="0.0 -1.0 0.0"/>
+  <axis xyz="-0.0 -0.0 -1.0"/>
 </joint>
 <joint name="Revolute 10" type="continuous">
-  <origin xyz="-0.4 -0.555 0.87" rpy="0 0 0"/>
+  <origin xyz="0.0 0.025965 0.876501" rpy="0 0 0"/>
   <parent link="base_link"/>
   <child link="leg_bl_1"/>
-  <axis xyz="0.0 -1.0 0.0"/>
+  <axis xyz="-0.0 -0.0 -1.0"/>
 </joint>
 <joint name="Revolute 11" type="continuous">
-  <origin xyz="0.37 0.535 0.87" rpy="0 0 0"/>
+  <origin xyz="0.77 1.115965 0.876501" rpy="0 0 0"/>
   <parent link="base_link"/>
   <child link="leg_fr_1"/>
-  <axis xyz="0.0 -1.0 0.0"/>
+  <axis xyz="-0.0 -0.0 -1.0"/>
 </joint>
 <joint name="Revolute 12" type="continuous">
-  <origin xyz="-0.4 0.535 0.87" rpy="0 0 0"/>
+  <origin xyz="0.0 1.115965 0.876501" rpy="0 0 0"/>
   <parent link="base_link"/>
   <child link="leg_fl_1"/>
-  <axis xyz="0.0 -1.0 0.0"/>
+  <axis xyz="-0.0 -0.0 -1.0"/>
 </joint>
 <joint name="Revolute 13" type="continuous">
@@ -212,5 +212,5 @@
   <parent link="leg_br_1"/>
   <child link="wheel_br_1"/>
-  <axis xyz="1.0 0.0 0.0"/>
+  <axis xyz="1.0 -0.0 -0.0"/>
 </joint>
 <joint name="Revolute 14" type="continuous">
@@ -218,5 +218,5 @@
   <parent link="leg_fr_1"/>
   <child link="wheel_fr_1"/>
-  <axis xyz="1.0 0.0 0.0"/>
+  <axis xyz="1.0 0.0 -0.0"/>
 </joint>
 <joint name="Revolute 15" type="continuous">
@@ -224,5 +224,5 @@
   <parent link="leg_bl_1"/>
   <child link="wheel_bl_1"/>
-  <axis xyz="-1.0 0.0 0.0"/>
+  <axis xyz="-1.0 -0.0 0.0"/>
 </joint>
 <joint name="Revolute 16" type="continuous">
@@ -230,5 +230,5 @@
   <parent link="leg_fl_1"/>
   <child link="wheel_fl_1"/>
-  <axis xyz="-1.0 0.0 0.0"/>
+  <axis xyz="-1.0 -0.0 0.0"/>
 </joint>
 </robot>

Commit message: update urdf

File: src/Rice_description/urdf/Rice.xacro (robot description, xacro)
@@ -6,5 +6,5 @@
 <link name="base_link">
   <inertial>
-    <origin xyz="0.38402832945911597 0.567977724226758 0.9197289790734344" rpy="0 0 0"/>
+    <origin xyz="0.38402832945911597 0.5679777242267577 0.9197289790734346" rpy="0 0 0"/>
     <mass value="111.52248073403698"/>
     <inertia ixx="19.278738" iyy="11.892444" izz="29.802061" ixy="0.058745" iyz="0.077376" ixz="0.004947"/>
@@ -26,5 +26,5 @@
 <link name="leg_br_1">
   <inertial>
-    <origin xyz="0.02067495895251792 0.05948901031816567 -0.42960523779205095" rpy="0 0 0"/>
+    <origin xyz="0.02067495895251803 0.05948901031816539 -0.4296052377920505" rpy="0 0 0"/>
     <mass value="19.428196282242897"/>
     <inertia ixx="0.69198" iyy="0.64895" izz="0.118365" ixy="-0.016967" iyz="-0.04479" ixz="-0.001759"/>
@@ -46,5 +46,5 @@
 <link name="leg_bl_1">
   <inertial>
-    <origin xyz="-0.020209424216131984 0.05818392702927147 -0.4348056527161479" rpy="0 0 0"/>
+    <origin xyz="-0.020209424216131908 0.05818392702927119 -0.43480565271614746" rpy="0 0 0"/>
     <mass value="19.9033372562808"/>
     <inertia ixx="0.720932" iyy="0.676639" izz="0.120784" ixy="0.017565" iyz="-0.050773" ixz="0.003917"/>
@@ -66,5 +66,5 @@
 <link name="leg_fr_1">
   <inertial>
-    <origin xyz="0.020209424438183965 -0.058184301381010606 -0.43480565196065807" rpy="0 0 0"/>
+    <origin xyz="0.020209424438183965 -0.058184301381010606 -0.4348056519606576" rpy="0 0 0"/>
     <mass value="19.90333719348541"/>
     <inertia ixx="0.720932" iyy="0.676639" izz="0.120784" ixy="0.017565" iyz="0.050773" ixz="-0.003917"/>
@@ -86,10 +86,10 @@
 <link name="leg_fl_1">
   <inertial>
-    <origin xyz="-0.020233756052453953 -0.058202816166196714 -0.4347330181911013" rpy="0 0 0"/>
+    <origin xyz="-0.02023375605245399 -0.058202816166196936 -0.4347330181911009" rpy="0 0 0"/>
     <mass value="19.897003188386865"/>
     <inertia ixx="0.72058" iyy="0.676271" izz="0.120724" ixy="-0.017537" iyz="0.050689" ixz="0.003807"/>
   </inertial>
   <visual>
-    <origin xyz="-0.0 -1.115965 -0.876501" rpy="0 0 0"/>
+    <origin xyz="0.0 -1.115965 -0.876501" rpy="0 0 0"/>
     <geometry>
       <mesh filename="file://$(find Rice_description)/meshes/leg_fl_1.stl" scale="0.001 0.001 0.001"/>
@@ -98,5 +98,5 @@
   </visual>
   <collision>
-    <origin xyz="-0.0 -1.115965 -0.876501" rpy="0 0 0"/>
+    <origin xyz="0.0 -1.115965 -0.876501" rpy="0 0 0"/>
     <geometry>
       <mesh filename="file://$(find Rice_description)/meshes/leg_fl_1.stl" scale="0.001 0.001 0.001"/>
@@ -106,7 +106,7 @@
 <link name="wheel_br_1">
   <inertial>
-    <origin xyz="-0.0036583592134993292 -1.8708468446995696e-07 4.2335822600381157e-07" rpy="0 0 0"/>
-    <mass value="65.80472593736363"/>
-    <inertia ixx="1.584128" iyy="0.836383" izz="0.836383" ixy="0.0" iyz="0.0" ixz="-0.0"/>
+    <origin xyz="-0.0036583592134993292 -1.8708468475445161e-07 4.2335822636463405e-07" rpy="0 0 0"/>
+    <mass value="65.80472593736363"/>
+    <inertia ixx="1.584128" iyy="0.836383" izz="0.836383" ixy="0.0" iyz="-0.0" ixz="-0.0"/>
   </inertial>
   <visual>
@@ -126,29 +126,29 @@
 <link name="wheel_fr_1">
   <inertial>
-    <origin xyz="-0.0036583592134961096 -1.8708470195250015e-07 4.233582252821666e-07" rpy="0 0 0"/>
+    <origin xyz="-0.0036583592134963316 -1.8708470239658936e-07 4.233582256152335e-07" rpy="0 0 0"/>
+    <mass value="65.80472593736363"/>
+    <inertia ixx="1.584128" iyy="0.836383" izz="0.836383" ixy="-0.0" iyz="-0.0" ixz="-0.0"/>
+  </inertial>
+  <visual>
+    <origin xyz="-0.863 -1.115965 -0.206501" rpy="0 0 0"/>
+    <geometry>
+      <mesh filename="file://$(find Rice_description)/meshes/wheel_fr_1.stl" scale="0.001 0.001 0.001"/>
+    </geometry>
+    <material name="silver"/>
+  </visual>
+  <collision>
+    <origin xyz="-0.863 -1.115965 -0.206501" rpy="0 0 0"/>
+    <geometry>
+      <mesh filename="file://$(find Rice_description)/meshes/wheel_fr_1.stl" scale="0.001 0.001 0.001"/>
+    </geometry>
+  </collision>
+</link>
+<link name="wheel_bl_1">
+  <inertial>
+    <origin xyz="0.0020000000000001406 -1.8708468407444e-07 4.233582261981006e-07" rpy="0 0 0"/>
     <mass value="65.80472593736363"/>
     <inertia ixx="1.584128" iyy="0.836383" izz="0.836383" ixy="-0.0" iyz="0.0" ixz="0.0"/>
   </inertial>
   <visual>
-    <origin xyz="-0.863 -1.115965 -0.206501" rpy="0 0 0"/>
-    <geometry>
-      <mesh filename="file://$(find Rice_description)/meshes/wheel_fr_1.stl" scale="0.001 0.001 0.001"/>
-    </geometry>
-    <material name="silver"/>
-  </visual>
-  <collision>
-    <origin xyz="-0.863 -1.115965 -0.206501" rpy="0 0 0"/>
-    <geometry>
-      <mesh filename="file://$(find Rice_description)/meshes/wheel_fr_1.stl" scale="0.001 0.001 0.001"/>
-    </geometry>
-  </collision>
-</link>
-<link name="wheel_bl_1">
-  <inertial>
-    <origin xyz="0.0020000000000000573 -1.870846836303508e-07 4.233582258372781e-07" rpy="0 0 0"/>
-    <mass value="65.80472593736363"/>
-    <inertia ixx="1.584128" iyy="0.836383" izz="0.836383" ixy="-0.0" iyz="0.0" ixz="0.0"/>
-  </inertial>
-  <visual>
     <origin xyz="0.093 -0.025965 -0.206501" rpy="0 0 0"/>
     <geometry>
@@ -166,5 +166,5 @@
 <link name="wheel_fl_1">
   <inertial>
-    <origin xyz="0.0020000000000037488 -1.8708469617934043e-07 4.2335822519889987e-07" rpy="0 0 0"/>
+    <origin xyz="0.0020000000000036933 -1.8708469684547424e-07 4.2335822555972236e-07" rpy="0 0 0"/>
     <mass value="65.80472593736363"/>
     <inertia ixx="1.584128" iyy="0.836383" izz="0.836383" ixy="0.0" iyz="0.0" ixz="0.0"/>
@@ -181,4 +181,44 @@
     <geometry>
       <mesh filename="file://$(find Rice_description)/meshes/wheel_fl_1.stl" scale="0.001 0.001 0.001"/>
+    </geometry>
+  </collision>
+</link>
+<link name="arm_1">
+  <inertial>
+    <origin xyz="-0.2584017090179747 0.002110884278794578 -0.07218880073119238" rpy="0 0 0"/>
+    <mass value="22.741450985256424"/>
+    <inertia ixx="1.72933" iyy="1.730341" izz="3.147968" ixy="0.000336" iyz="0.000291" ixz="-0.001081"/>
+  </inertial>
+  <visual>
+    <origin xyz="-0.6435 -0.570965 -0.873501" rpy="0 0 0"/>
+    <geometry>
+      <mesh filename="file://$(find Rice_description)/meshes/arm_1.stl" scale="0.001 0.001 0.001"/>
+    </geometry>
+    <material name="silver"/>
+  </visual>
+  <collision>
+    <origin xyz="-0.6435 -0.570965 -0.873501" rpy="0 0 0"/>
+    <geometry>
+      <mesh filename="file://$(find Rice_description)/meshes/arm_1.stl" scale="0.001 0.001 0.001"/>
+    </geometry>
+  </collision>
+</link>
+<link name="solar_1">
+  <inertial>
+    <origin xyz="4.377609386096992e-13 0.39349657074105626 0.24368297346942225" rpy="0 0 0"/>
+    <mass value="131.93512225473023"/>
+    <inertia ixx="26.841833" iyy="21.913769" izz="48.508633" ixy="-0.0" iyz="-6.5e-05" ixz="0.0"/>
+  </inertial>
+  <visual>
+    <origin xyz="-0.385 -0.177463 -0.982466" rpy="0 0 0"/>
+    <geometry>
+      <mesh filename="file://$(find Rice_description)/meshes/solar_1.stl" scale="0.001 0.001 0.001"/>
+    </geometry>
+    <material name="silver"/>
+  </visual>
+  <collision>
+    <origin xyz="-0.385 -0.177463 -0.982466" rpy="0 0 0"/>
+    <geometry>
+      <mesh filename="file://$(find Rice_description)/meshes/solar_1.stl" scale="0.001 0.001 0.001"/>
     </geometry>
   </collision>
@@ -212,5 +252,5 @@
   <parent link="leg_br_1"/>
   <child link="wheel_br_1"/>
-  <axis xyz="1.0 -0.0 -0.0"/>
+  <axis xyz="1.0 0.0 -0.0"/>
 </joint>
 <joint name="Revolute 14" type="continuous">
@@ -232,3 +272,13 @@
   <axis xyz="-1.0 -0.0 0.0"/>
 </joint>
+<joint name="Rigid 17" type="fixed">
+  <origin xyz="0.6435 0.570965 0.873501" rpy="0 0 0"/>
+  <parent link="base_link"/>
+  <child link="arm_1"/>
+</joint>
+<joint name="Rigid 18" type="fixed">
+  <origin xyz="0.385 0.177463 0.982466" rpy="0 0 0"/>
+  <parent link="base_link"/>
+  <child link="solar_1"/>
+</joint>
 </robot>
