Commit message: update urdf

File: src/Rice_description/urdf/Rice.xacro (robot description, xacro)
@@ -6,5 +6,5 @@
 <link name="base_link">
   <inertial>
-    <origin xyz="0.38402832945911597 0.5679777242267577 0.9197289790734346" rpy="0 0 0"/>
+    <origin xyz="0.38402832945911586 0.2840129113114328 1.0082275557152205" rpy="0 0 0"/>
     <mass value="111.52248073403698"/>
     <inertia ixx="19.278738" iyy="11.892444" izz="29.802061" ixy="0.058745" iyz="0.077376" ixz="0.004947"/>
@@ -24,261 +24,261 @@
   </collision>
 </link>
-<link name="leg_br_1">
-  <inertial>
-    <origin xyz="0.02067495895251803 0.05948901031816539 -0.4296052377920505" rpy="0 0 0"/>
+<link name="leg_bl_2">
+  <inertial>
+    <origin xyz="-0.020209424216131974 0.058184114113957186 -0.43480607607437316" rpy="0 0 0"/>
+    <mass value="19.9033372562808"/>
+    <inertia ixx="0.720932" iyy="0.676639" izz="0.120784" ixy="0.017565" iyz="-0.050773" ixz="0.003917"/>
+  </inertial>
+  <visual>
+    <origin xyz="0.0 0.258 -0.965" rpy="0 0 0"/>
+    <geometry>
+      <mesh filename="file://$(find Rice_description)/meshes/leg_bl_2.stl" scale="0.001 0.001 0.001"/>
+    </geometry>
+    <material name="silver"/>
+  </visual>
+  <collision>
+    <origin xyz="0.0 0.258 -0.965" rpy="0 0 0"/>
+    <geometry>
+      <mesh filename="file://$(find Rice_description)/meshes/leg_bl_2.stl" scale="0.001 0.001 0.001"/>
+    </geometry>
+  </collision>
+</link>
+<link name="leg_br_2">
+  <inertial>
+    <origin xyz="0.020674958952517808 0.059489197402851246 -0.4296056611502763" rpy="0 0 0"/>
     <mass value="19.428196282242897"/>
     <inertia ixx="0.69198" iyy="0.64895" izz="0.118365" ixy="-0.016967" iyz="-0.04479" ixz="-0.001759"/>
   </inertial>
   <visual>
-    <origin xyz="-0.77 -0.025965 -0.876501" rpy="0 0 0"/>
-    <geometry>
-      <mesh filename="file://$(find Rice_description)/meshes/leg_br_1.stl" scale="0.001 0.001 0.001"/>
-    </geometry>
-    <material name="silver"/>
-  </visual>
-  <collision>
-    <origin xyz="-0.77 -0.025965 -0.876501" rpy="0 0 0"/>
-    <geometry>
-      <mesh filename="file://$(find Rice_description)/meshes/leg_br_1.stl" scale="0.001 0.001 0.001"/>
-    </geometry>
-  </collision>
-</link>
-<link name="leg_bl_1">
-  <inertial>
-    <origin xyz="-0.020209424216131908 0.05818392702927119 -0.43480565271614746" rpy="0 0 0"/>
-    <mass value="19.9033372562808"/>
-    <inertia ixx="0.720932" iyy="0.676639" izz="0.120784" ixy="0.017565" iyz="-0.050773" ixz="0.003917"/>
-  </inertial>
-  <visual>
-    <origin xyz="-0.0 -0.025965 -0.876501" rpy="0 0 0"/>
-    <geometry>
-      <mesh filename="file://$(find Rice_description)/meshes/leg_bl_1.stl" scale="0.001 0.001 0.001"/>
-    </geometry>
-    <material name="silver"/>
-  </visual>
-  <collision>
-    <origin xyz="-0.0 -0.025965 -0.876501" rpy="0 0 0"/>
-    <geometry>
-      <mesh filename="file://$(find Rice_description)/meshes/leg_bl_1.stl" scale="0.001 0.001 0.001"/>
-    </geometry>
-  </collision>
-</link>
-<link name="leg_fr_1">
-  <inertial>
-    <origin xyz="0.020209424438183965 -0.058184301381010606 -0.4348056519606576" rpy="0 0 0"/>
+    <origin xyz="-0.77 0.258 -0.965" rpy="0 0 0"/>
+    <geometry>
+      <mesh filename="file://$(find Rice_description)/meshes/leg_br_2.stl" scale="0.001 0.001 0.001"/>
+    </geometry>
+    <material name="silver"/>
+  </visual>
+  <collision>
+    <origin xyz="-0.77 0.258 -0.965" rpy="0 0 0"/>
+    <geometry>
+      <mesh filename="file://$(find Rice_description)/meshes/leg_br_2.stl" scale="0.001 0.001 0.001"/>
+    </geometry>
+  </collision>
+</link>
+<link name="leg_fl_2">
+  <inertial>
+    <origin xyz="-0.020233756052453943 -0.05820262908151064 -0.43473344154930404" rpy="0 0 0"/>
+    <mass value="19.897003188386865"/>
+    <inertia ixx="0.72058" iyy="0.676271" izz="0.120724" ixy="-0.017537" iyz="0.050689" ixz="0.003807"/>
+  </inertial>
+  <visual>
+    <origin xyz="0.0 -0.832 -0.965" rpy="0 0 0"/>
+    <geometry>
+      <mesh filename="file://$(find Rice_description)/meshes/leg_fl_2.stl" scale="0.001 0.001 0.001"/>
+    </geometry>
+    <material name="silver"/>
+  </visual>
+  <collision>
+    <origin xyz="0.0 -0.832 -0.965" rpy="0 0 0"/>
+    <geometry>
+      <mesh filename="file://$(find Rice_description)/meshes/leg_fl_2.stl" scale="0.001 0.001 0.001"/>
+    </geometry>
+  </collision>
+</link>
+<link name="leg_fr_2">
+  <inertial>
+    <origin xyz="0.020209424438183632 -0.05818411429632453 -0.43480607531886073" rpy="0 0 0"/>
     <mass value="19.90333719348541"/>
     <inertia ixx="0.720932" iyy="0.676639" izz="0.120784" ixy="0.017565" iyz="0.050773" ixz="-0.003917"/>
   </inertial>
   <visual>
-    <origin xyz="-0.77 -1.115965 -0.876501" rpy="0 0 0"/>
-    <geometry>
-      <mesh filename="file://$(find Rice_description)/meshes/leg_fr_1.stl" scale="0.001 0.001 0.001"/>
-    </geometry>
-    <material name="silver"/>
-  </visual>
-  <collision>
-    <origin xyz="-0.77 -1.115965 -0.876501" rpy="0 0 0"/>
-    <geometry>
-      <mesh filename="file://$(find Rice_description)/meshes/leg_fr_1.stl" scale="0.001 0.001 0.001"/>
-    </geometry>
-  </collision>
-</link>
-<link name="leg_fl_1">
-  <inertial>
-    <origin xyz="-0.02023375605245399 -0.058202816166196936 -0.4347330181911009" rpy="0 0 0"/>
-    <mass value="19.897003188386865"/>
-    <inertia ixx="0.72058" iyy="0.676271" izz="0.120724" ixy="-0.017537" iyz="0.050689" ixz="0.003807"/>
-  </inertial>
-  <visual>
-    <origin xyz="0.0 -1.115965 -0.876501" rpy="0 0 0"/>
-    <geometry>
-      <mesh filename="file://$(find Rice_description)/meshes/leg_fl_1.stl" scale="0.001 0.001 0.001"/>
-    </geometry>
-    <material name="silver"/>
-  </visual>
-  <collision>
-    <origin xyz="0.0 -1.115965 -0.876501" rpy="0 0 0"/>
-    <geometry>
-      <mesh filename="file://$(find Rice_description)/meshes/leg_fl_1.stl" scale="0.001 0.001 0.001"/>
-    </geometry>
-  </collision>
-</link>
-<link name="wheel_br_1">
-  <inertial>
-    <origin xyz="-0.0036583592134993292 -1.8708468475445161e-07 4.2335822636463405e-07" rpy="0 0 0"/>
-    <mass value="65.80472593736363"/>
-    <inertia ixx="1.584128" iyy="0.836383" izz="0.836383" ixy="0.0" iyz="-0.0" ixz="-0.0"/>
-  </inertial>
-  <visual>
-    <origin xyz="-0.863 -0.025965 -0.206501" rpy="0 0 0"/>
-    <geometry>
-      <mesh filename="file://$(find Rice_description)/meshes/wheel_br_1.stl" scale="0.001 0.001 0.001"/>
-    </geometry>
-    <material name="silver"/>
-  </visual>
-  <collision>
-    <origin xyz="-0.863 -0.025965 -0.206501" rpy="0 0 0"/>
-    <geometry>
-      <mesh filename="file://$(find Rice_description)/meshes/wheel_br_1.stl" scale="0.001 0.001 0.001"/>
-    </geometry>
-  </collision>
-</link>
-<link name="wheel_fr_1">
-  <inertial>
-    <origin xyz="-0.0036583592134963316 -1.8708470239658936e-07 4.233582256152335e-07" rpy="0 0 0"/>
-    <mass value="65.80472593736363"/>
-    <inertia ixx="1.584128" iyy="0.836383" izz="0.836383" ixy="-0.0" iyz="-0.0" ixz="-0.0"/>
-  </inertial>
-  <visual>
-    <origin xyz="-0.863 -1.115965 -0.206501" rpy="0 0 0"/>
-    <geometry>
-      <mesh filename="file://$(find Rice_description)/meshes/wheel_fr_1.stl" scale="0.001 0.001 0.001"/>
-    </geometry>
-    <material name="silver"/>
-  </visual>
-  <collision>
-    <origin xyz="-0.863 -1.115965 -0.206501" rpy="0 0 0"/>
-    <geometry>
-      <mesh filename="file://$(find Rice_description)/meshes/wheel_fr_1.stl" scale="0.001 0.001 0.001"/>
-    </geometry>
-  </collision>
-</link>
-<link name="wheel_bl_1">
-  <inertial>
-    <origin xyz="0.0020000000000001406 -1.8708468407444e-07 4.233582261981006e-07" rpy="0 0 0"/>
+    <origin xyz="-0.77 -0.832 -0.965" rpy="0 0 0"/>
+    <geometry>
+      <mesh filename="file://$(find Rice_description)/meshes/leg_fr_2.stl" scale="0.001 0.001 0.001"/>
+    </geometry>
+    <material name="silver"/>
+  </visual>
+  <collision>
+    <origin xyz="-0.77 -0.832 -0.965" rpy="0 0 0"/>
+    <geometry>
+      <mesh filename="file://$(find Rice_description)/meshes/leg_fr_2.stl" scale="0.001 0.001 0.001"/>
+    </geometry>
+  </collision>
+</link>
+<link name="wheel_br_2">
+  <inertial>
+    <origin xyz="-0.00200000000000089 7.66053886991358e-15 -1.4432899320127035e-15" rpy="0 0 0"/>
+    <mass value="65.80472593736363"/>
+    <inertia ixx="1.584128" iyy="0.836383" izz="0.836383" ixy="0.0" iyz="0.0" ixz="0.0"/>
+  </inertial>
+  <visual>
+    <origin xyz="-0.862 0.258 -0.295" rpy="0 0 0"/>
+    <geometry>
+      <mesh filename="file://$(find Rice_description)/meshes/wheel_br_2.stl" scale="0.001 0.001 0.001"/>
+    </geometry>
+    <material name="silver"/>
+  </visual>
+  <collision>
+    <origin xyz="-0.862 0.258 -0.295" rpy="0 0 0"/>
+    <geometry>
+      <mesh filename="file://$(find Rice_description)/meshes/wheel_br_2.stl" scale="0.001 0.001 0.001"/>
+    </geometry>
+  </collision>
+</link>
+<link name="wheel_fr_2">
+  <inertial>
+    <origin xyz="-0.001999999999996671 -1.0547118733938987e-14 2.325917236589703e-14" rpy="0 0 0"/>
+    <mass value="65.80472593736363"/>
+    <inertia ixx="1.584128" iyy="0.836383" izz="0.836383" ixy="-0.0" iyz="0.0" ixz="-0.0"/>
+  </inertial>
+  <visual>
+    <origin xyz="-0.862 -0.832 -0.295" rpy="0 0 0"/>
+    <geometry>
+      <mesh filename="file://$(find Rice_description)/meshes/wheel_fr_2.stl" scale="0.001 0.001 0.001"/>
+    </geometry>
+    <material name="silver"/>
+  </visual>
+  <collision>
+    <origin xyz="-0.862 -0.832 -0.295" rpy="0 0 0"/>
+    <geometry>
+      <mesh filename="file://$(find Rice_description)/meshes/wheel_fr_2.stl" scale="0.001 0.001 0.001"/>
+    </geometry>
+  </collision>
+</link>
+<link name="wheel_fl_2">
+  <inertial>
+    <origin xyz="0.00200000000000386 -4.6629367034256575e-15 2.3370194668359545e-14" rpy="0 0 0"/>
+    <mass value="65.80472593736363"/>
+    <inertia ixx="1.584128" iyy="0.836383" izz="0.836383" ixy="0.0" iyz="-0.0" ixz="0.0"/>
+  </inertial>
+  <visual>
+    <origin xyz="0.092 -0.832 -0.295" rpy="0 0 0"/>
+    <geometry>
+      <mesh filename="file://$(find Rice_description)/meshes/wheel_fl_2.stl" scale="0.001 0.001 0.001"/>
+    </geometry>
+    <material name="silver"/>
+  </visual>
+  <collision>
+    <origin xyz="0.092 -0.832 -0.295" rpy="0 0 0"/>
+    <geometry>
+      <mesh filename="file://$(find Rice_description)/meshes/wheel_fl_2.stl" scale="0.001 0.001 0.001"/>
+    </geometry>
+  </collision>
+</link>
+<link name="wheel_bl_2">
+  <inertial>
+    <origin xyz="0.001999999999999974 7.605027718682322e-15 -1.5543122344752192e-15" rpy="0 0 0"/>
     <mass value="65.80472593736363"/>
     <inertia ixx="1.584128" iyy="0.836383" izz="0.836383" ixy="-0.0" iyz="0.0" ixz="0.0"/>
   </inertial>
   <visual>
-    <origin xyz="0.093 -0.025965 -0.206501" rpy="0 0 0"/>
-    <geometry>
-      <mesh filename="file://$(find Rice_description)/meshes/wheel_bl_1.stl" scale="0.001 0.001 0.001"/>
-    </geometry>
-    <material name="silver"/>
-  </visual>
-  <collision>
-    <origin xyz="0.093 -0.025965 -0.206501" rpy="0 0 0"/>
-    <geometry>
-      <mesh filename="file://$(find Rice_description)/meshes/wheel_bl_1.stl" scale="0.001 0.001 0.001"/>
-    </geometry>
-  </collision>
-</link>
-<link name="wheel_fl_1">
-  <inertial>
-    <origin xyz="0.0020000000000036933 -1.8708469684547424e-07 4.2335822555972236e-07" rpy="0 0 0"/>
-    <mass value="65.80472593736363"/>
-    <inertia ixx="1.584128" iyy="0.836383" izz="0.836383" ixy="0.0" iyz="0.0" ixz="0.0"/>
-  </inertial>
-  <visual>
-    <origin xyz="0.093 -1.115965 -0.206501" rpy="0 0 0"/>
-    <geometry>
-      <mesh filename="file://$(find Rice_description)/meshes/wheel_fl_1.stl" scale="0.001 0.001 0.001"/>
-    </geometry>
-    <material name="silver"/>
-  </visual>
-  <collision>
-    <origin xyz="0.093 -1.115965 -0.206501" rpy="0 0 0"/>
-    <geometry>
-      <mesh filename="file://$(find Rice_description)/meshes/wheel_fl_1.stl" scale="0.001 0.001 0.001"/>
-    </geometry>
-  </collision>
-</link>
-<link name="arm_1">
-  <inertial>
-    <origin xyz="-0.2584017090179747 0.002110884278794578 -0.07218880073119238" rpy="0 0 0"/>
+    <origin xyz="0.092 0.258 -0.295" rpy="0 0 0"/>
+    <geometry>
+      <mesh filename="file://$(find Rice_description)/meshes/wheel_bl_2.stl" scale="0.001 0.001 0.001"/>
+    </geometry>
+    <material name="silver"/>
+  </visual>
+  <collision>
+    <origin xyz="0.092 0.258 -0.295" rpy="0 0 0"/>
+    <geometry>
+      <mesh filename="file://$(find Rice_description)/meshes/wheel_bl_2.stl" scale="0.001 0.001 0.001"/>
+    </geometry>
+  </collision>
+</link>
+<link name="arm_2">
+  <inertial>
+    <origin xyz="0.12774204119968946 -0.22461184977364618 -0.07218922408939565" rpy="0 0 0"/>
     <mass value="22.741450985256424"/>
     <inertia ixx="1.72933" iyy="1.730341" izz="3.147968" ixy="0.000336" iyz="0.000291" ixz="-0.001081"/>
   </inertial>
   <visual>
-    <origin xyz="-0.6435 -0.570965 -0.873501" rpy="0 0 0"/>
-    <geometry>
-      <mesh filename="file://$(find Rice_description)/meshes/arm_1.stl" scale="0.001 0.001 0.001"/>
-    </geometry>
-    <material name="silver"/>
-  </visual>
-  <collision>
-    <origin xyz="-0.6435 -0.570965 -0.873501" rpy="0 0 0"/>
-    <geometry>
-      <mesh filename="file://$(find Rice_description)/meshes/arm_1.stl" scale="0.001 0.001 0.001"/>
-    </geometry>
-  </collision>
-</link>
-<link name="solar_1">
-  <inertial>
-    <origin xyz="4.377609386096992e-13 0.39349657074105626 0.24368297346942225" rpy="0 0 0"/>
+    <origin xyz="-0.25575 -0.510868 -0.962" rpy="0 0 0"/>
+    <geometry>
+      <mesh filename="file://$(find Rice_description)/meshes/arm_2.stl" scale="0.001 0.001 0.001"/>
+    </geometry>
+    <material name="silver"/>
+  </visual>
+  <collision>
+    <origin xyz="-0.25575 -0.510868 -0.962" rpy="0 0 0"/>
+    <geometry>
+      <mesh filename="file://$(find Rice_description)/meshes/arm_2.stl" scale="0.001 0.001 0.001"/>
+    </geometry>
+  </collision>
+</link>
+<link name="solar_2">
+  <inertial>
+    <origin xyz="4.3731684939984916e-13 0.48199475782572393 0.5276475501112076" rpy="0 0 0"/>
     <mass value="131.93512225473023"/>
     <inertia ixx="26.841833" iyy="21.913769" izz="48.508633" ixy="-0.0" iyz="-6.5e-05" ixz="0.0"/>
   </inertial>
   <visual>
-    <origin xyz="-0.385 -0.177463 -0.982466" rpy="0 0 0"/>
-    <geometry>
-      <mesh filename="file://$(find Rice_description)/meshes/solar_1.stl" scale="0.001 0.001 0.001"/>
-    </geometry>
-    <material name="silver"/>
-  </visual>
-  <collision>
-    <origin xyz="-0.385 -0.177463 -0.982466" rpy="0 0 0"/>
-    <geometry>
-      <mesh filename="file://$(find Rice_description)/meshes/solar_1.stl" scale="0.001 0.001 0.001"/>
-    </geometry>
-  </collision>
-</link>
-<joint name="Revolute 9" type="continuous">
-  <origin xyz="0.77 0.025965 0.876501" rpy="0 0 0"/>
-  <parent link="base_link"/>
-  <child link="leg_br_1"/>
-  <axis xyz="-0.0 -0.0 -1.0"/>
-</joint>
-<joint name="Revolute 10" type="continuous">
-  <origin xyz="0.0 0.025965 0.876501" rpy="0 0 0"/>
-  <parent link="base_link"/>
-  <child link="leg_bl_1"/>
-  <axis xyz="-0.0 -0.0 -1.0"/>
-</joint>
-<joint name="Revolute 11" type="continuous">
-  <origin xyz="0.77 1.115965 0.876501" rpy="0 0 0"/>
-  <parent link="base_link"/>
-  <child link="leg_fr_1"/>
-  <axis xyz="-0.0 -0.0 -1.0"/>
-</joint>
-<joint name="Revolute 12" type="continuous">
-  <origin xyz="0.0 1.115965 0.876501" rpy="0 0 0"/>
-  <parent link="base_link"/>
-  <child link="leg_fl_1"/>
-  <axis xyz="-0.0 -0.0 -1.0"/>
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