Commit message: Update robotpadi.xacro

File: src/robotpadi_description/urdf/robotpadi.xacro (robot description, xacro)
@@ -6,5 +6,5 @@
 <link name="base_link">
   <inertial>
-    <origin xyz="2.4824220796767777 0.28115799017238796 1.0082275557140772" rpy="0 0 0"/>
+    <origin xyz="0.38402832945911336 0.2840129113095087 1.0082275557140674" rpy="0 0 0"/>
     <mass value="111.52248073403693"/>
     <inertia ixx="19.278738" iyy="11.892444" izz="29.802061" ixy="0.058745" iyz="0.077376" ixz="0.004947"/>
@@ -26,10 +26,10 @@
 <link name="fr_steering_1">
   <inertial>
-    <origin xyz="0.020209174655847928 -0.05818403543565476 -0.43480607532017557" rpy="0 0 0"/>
+    <origin xyz="0.020209424438183965 -0.058184114298542866 -0.434806075320194" rpy="0 0 0"/>
     <mass value="19.903337193485434"/>
     <inertia ixx="0.720932" iyy="0.676639" izz="0.120784" ixy="0.017565" iyz="0.050773" ixz="-0.003917"/>
   </inertial>
   <visual>
-    <origin xyz="-2.868394 -0.829145 -0.965" rpy="0 0 0"/>
+    <origin xyz="-0.77 -0.832 -0.965" rpy="0 0 0"/>
     <geometry>
       <mesh filename="file://$(find robotpadi_description)/meshes/fr_steering_1.stl" scale="0.001 0.001 0.001"/>
@@ -38,5 +38,5 @@
   </visual>
   <collision>
-    <origin xyz="-2.868394 -0.829145 -0.965" rpy="0 0 0"/>
+    <origin xyz="-0.77 -0.832 -0.965" rpy="0 0 0"/>
     <geometry>
       <mesh filename="file://$(find robotpadi_description)/meshes/fr_steering_1.stl" scale="0.001 0.001 0.001"/>
@@ -46,10 +46,10 @@
 <link name="br_steering_1">
   <inertial>
-    <origin xyz="0.02067470917018399 0.05948927608269658 -0.4296056612602748" rpy="0 0 0"/>
+    <origin xyz="0.02067495895252003 0.05948919721980847 -0.42960566126027544" rpy="0 0 0"/>
     <mass value="19.42819628224292"/>
     <inertia ixx="0.69198" iyy="0.64895" izz="0.118365" ixy="-0.016967" iyz="-0.04479" ixz="-0.001759"/>
   </inertial>
   <visual>
-    <origin xyz="-2.868394 0.260855 -0.965" rpy="0 0 0"/>
+    <origin xyz="-0.77 0.258 -0.965" rpy="0 0 0"/>
     <geometry>
       <mesh filename="file://$(find robotpadi_description)/meshes/br_steering_1.stl" scale="0.001 0.001 0.001"/>
@@ -58,5 +58,5 @@
   </visual>
   <collision>
-    <origin xyz="-2.868394 0.260855 -0.965" rpy="0 0 0"/>
+    <origin xyz="-0.77 0.258 -0.965" rpy="0 0 0"/>
     <geometry>
       <mesh filename="file://$(find robotpadi_description)/meshes/br_steering_1.stl" scale="0.001 0.001 0.001"/>
@@ -66,10 +66,10 @@
 <link name="fl_steering_1">
   <inertial>
-    <origin xyz="-0.020675208734855843 -0.059489118356931936 -0.4296056612602346" rpy="0 0 0"/>
+    <origin xyz="-0.02067495895252023 -0.05948919721981982 -0.42960566126025335" rpy="0 0 0"/>
     <mass value="19.42819628224292"/>
     <inertia ixx="0.69198" iyy="0.64895" izz="0.118365" ixy="-0.016967" iyz="0.04479" ixz="0.001759"/>
   </inertial>
   <visual>
-    <origin xyz="-2.098394 -0.829145 -0.965" rpy="0 0 0"/>
+    <origin xyz="0.0 -0.832 -0.965" rpy="0 0 0"/>
     <geometry>
       <mesh filename="file://$(find robotpadi_description)/meshes/fl_steering_1.stl" scale="0.001 0.001 0.001"/>
@@ -78,5 +78,5 @@
   </visual>
   <collision>
-    <origin xyz="-2.098394 -0.829145 -0.965" rpy="0 0 0"/>
+    <origin xyz="0.0 -0.832 -0.965" rpy="0 0 0"/>
     <geometry>
       <mesh filename="file://$(find robotpadi_description)/meshes/fl_steering_1.stl" scale="0.001 0.001 0.001"/>
@@ -86,10 +86,10 @@
 <link name="bl_steering_1">
   <inertial>
-    <origin xyz="-0.020209674220515783 0.058184193161417125 -0.4348060753202152" rpy="0 0 0"/>
+    <origin xyz="-0.02020942443818015 0.05818411429852913 -0.4348060753202161" rpy="0 0 0"/>
     <mass value="19.903337193485434"/>
     <inertia ixx="0.720932" iyy="0.676639" izz="0.120784" ixy="0.017565" iyz="-0.050773" ixz="0.003917"/>
   </inertial>
   <visual>
-    <origin xyz="-2.098394 0.260855 -0.965" rpy="0 0 0"/>
+    <origin xyz="0.0 0.258 -0.965" rpy="0 0 0"/>
     <geometry>
       <mesh filename="file://$(find robotpadi_description)/meshes/bl_steering_1.stl" scale="0.001 0.001 0.001"/>
@@ -98,5 +98,5 @@
   </visual>
   <collision>
-    <origin xyz="-2.098394 0.260855 -0.965" rpy="0 0 0"/>
+    <origin xyz="0.0 0.258 -0.965" rpy="0 0 0"/>
     <geometry>
       <mesh filename="file://$(find robotpadi_description)/meshes/bl_steering_1.stl" scale="0.001 0.001 0.001"/>
@@ -106,10 +106,10 @@
 <link name="br_wheel_1">
   <inertial>
-    <origin xyz="0.00199975021766452 7.886290126490891e-08 -9.992007221626409e-16" rpy="0 0 0"/>
-    <mass value="65.80472593736373"/>
-    <inertia ixx="1.584128" iyy="0.836383" izz="0.836383" ixy="0.0" iyz="0.0" ixz="0.0"/>
-  </inertial>
-  <visual>
-    <origin xyz="-2.956394 0.260855 -0.295" rpy="0 0 0"/>
+    <origin xyz="0.002000000000001445 8.992806499463768e-15 -8.326672684688674e-16" rpy="0 0 0"/>
+    <mass value="65.80472593736373"/>
+    <inertia ixx="1.584128" iyy="0.836383" izz="0.836383" ixy="0.0" iyz="0.0" ixz="0.0"/>
+  </inertial>
+  <visual>
+    <origin xyz="-0.858 0.258 -0.295" rpy="0 0 0"/>
     <geometry>
       <mesh filename="file://$(find robotpadi_description)/meshes/br_wheel_1.stl" scale="0.001 0.001 0.001"/>
@@ -118,5 +118,5 @@
   </visual>
   <collision>
-    <origin xyz="-2.956394 0.260855 -0.295" rpy="0 0 0"/>
+    <origin xyz="-0.858 0.258 -0.295" rpy="0 0 0"/>
     <geometry>
       <mesh filename="file://$(find robotpadi_description)/meshes/br_wheel_1.stl" scale="0.001 0.001 0.001"/>
@@ -126,10 +126,10 @@
 <link name="fl_wheel_1">
   <inertial>
-    <origin xyz="-0.0020002497823359278 7.886288377889628e-08 4.368727601899991e-14" rpy="0 0 0"/>
-    <mass value="65.80472593736373"/>
-    <inertia ixx="1.584128" iyy="0.836383" izz="0.836383" ixy="0.0" iyz="0.0" ixz="0.0"/>
-  </inertial>
-  <visual>
-    <origin xyz="-2.010394 -0.829145 -0.295" rpy="0 0 0"/>
+    <origin xyz="-0.0020000000000005708 -8.770761894538737e-15 2.398081733190338e-14" rpy="0 0 0"/>
+    <mass value="65.80472593736373"/>
+    <inertia ixx="1.584128" iyy="0.836383" izz="0.836383" ixy="0.0" iyz="0.0" ixz="0.0"/>
+  </inertial>
+  <visual>
+    <origin xyz="0.088 -0.832 -0.295" rpy="0 0 0"/>
     <geometry>
       <mesh filename="file://$(find robotpadi_description)/meshes/fl_wheel_1.stl" scale="0.001 0.001 0.001"/>
@@ -138,5 +138,5 @@
   </visual>
   <collision>
-    <origin xyz="-2.010394 -0.829145 -0.295" rpy="0 0 0"/>
+    <origin xyz="0.088 -0.832 -0.295" rpy="0 0 0"/>
     <geometry>
       <mesh filename="file://$(find robotpadi_description)/meshes/fl_wheel_1.stl" scale="0.001 0.001 0.001"/>
@@ -146,10 +146,10 @@
 <link name="bl_wheel_1">
   <inertial>
-    <origin xyz="-0.002000249782336372 7.886288388991858e-08 -7.771561172376096e-16" rpy="0 0 0"/>
-    <mass value="65.80472593736373"/>
-    <inertia ixx="1.584128" iyy="0.836383" izz="0.836383" ixy="0.0" iyz="0.0" ixz="0.0"/>
-  </inertial>
-  <visual>
-    <origin xyz="-2.010394 0.260855 -0.295" rpy="0 0 0"/>
+    <origin xyz="-0.002000000000001237 -8.493206138382448e-15 -6.661338147750939e-16" rpy="0 0 0"/>
+    <mass value="65.80472593736373"/>
+    <inertia ixx="1.584128" iyy="0.836383" izz="0.836383" ixy="0.0" iyz="0.0" ixz="0.0"/>
+  </inertial>
+  <visual>
+    <origin xyz="0.088 0.258 -0.295" rpy="0 0 0"/>
     <geometry>
       <mesh filename="file://$(find robotpadi_description)/meshes/bl_wheel_1.stl" scale="0.001 0.001 0.001"/>
@@ -158,5 +158,5 @@
   </visual>
   <collision>
-    <origin xyz="-2.010394 0.260855 -0.295" rpy="0 0 0"/>
+    <origin xyz="0.088 0.258 -0.295" rpy="0 0 0"/>
     <geometry>
       <mesh filename="file://$(find robotpadi_description)/meshes/bl_wheel_1.stl" scale="0.001 0.001 0.001"/>
@@ -166,10 +166,10 @@
 <link name="fr_wheel_1">
   <inertial>
-    <origin xyz="0.0019997502176680726 7.886289754566178e-08 4.340972026284362e-14" rpy="0 0 0"/>
-    <mass value="65.80472593736373"/>
-    <inertia ixx="1.584128" iyy="0.836383" izz="0.836383" ixy="0.0" iyz="0.0" ixz="0.0"/>
-  </inertial>
-  <visual>
-    <origin xyz="-2.956394 -0.829145 -0.295" rpy="0 0 0"/>
+    <origin xyz="0.0019999999999994467 7.549516567451064e-15 2.4313884239290928e-14" rpy="0 0 0"/>
+    <mass value="65.80472593736373"/>
+    <inertia ixx="1.584128" iyy="0.836383" izz="0.836383" ixy="0.0" iyz="0.0" ixz="0.0"/>
+  </inertial>
+  <visual>
+    <origin xyz="-0.858 -0.832 -0.295" rpy="0 0 0"/>
     <geometry>
       <mesh filename="file://$(find robotpadi_description)/meshes/fr_wheel_1.stl" scale="0.001 0.001 0.001"/>
@@ -178,5 +178,5 @@
   </visual>
   <collision>
-    <origin xyz="-2.956394 -0.829145 -0.295" rpy="0 0 0"/>
+    <origin xyz="-0.858 -0.832 -0.295" rpy="0 0 0"/>
     <geometry>
       <mesh filename="file://$(find robotpadi_description)/meshes/fr_wheel_1.stl" scale="0.001 0.001 0.001"/>
@@ -186,10 +186,10 @@
 <link name="panel_1">
   <inertial>
-    <origin xyz="-2.098394249781907 0.002849836688600116 0.2876475501112252" rpy="0 0 0"/>
+    <origin xyz="4.287126209590042e-13 -5.242174278385914e-06 0.287647550111215" rpy="0 0 0"/>
     <mass value="131.93512225471943"/>
     <inertia ixx="26.841833" iyy="21.913769" izz="48.508633" ixy="0.0" iyz="-6.5e-05" ixz="0.0"/>
   </inertial>
   <visual>
-    <origin xyz="-4.581788 -0.28129 -1.027" rpy="0 0 0"/>
+    <origin xyz="-0.385 -0.287 -1.027" rpy="0 0 0"/>
     <geometry>
       <mesh filename="file://$(find robotpadi_description)/meshes/panel_1.stl" scale="0.001 0.001 0.001"/>
@@ -198,5 +198,5 @@
   </visual>
   <collision>
-    <origin xyz="-4.581788 -0.28129 -1.027" rpy="0 0 0"/>
+    <origin xyz="-0.385 -0.287 -1.027" rpy="0 0 0"/>
     <geometry>
       <mesh filename="file://$(find robotpadi_description)/meshes/panel_1.stl" scale="0.001 0.001 0.001"/>
@@ -206,10 +206,10 @@
 <link name="arm_1">
   <inertial>
-    <origin xyz="-0.2584019710100889 0.0021111539984787764 -0.07218922154686003" rpy="0 0 0"/>
+    <origin xyz="-0.2584017212277529 0.0021110751355971624 -0.07218922154687024" rpy="0 0 0"/>
     <mass value="22.7414514992095"/>
     <inertia ixx="1.72933" iyy="1.730341" izz="3.147968" ixy="0.000336" iyz="0.000291" ixz="-0.001081"/>
   </inertial>
   <visual>
-    <origin xyz="-2.741894 -0.284145 -0.962" rpy="0 0 0"/>
+    <origin xyz="-0.6435 -0.287 -0.962" rpy="0 0 0"/>
     <geometry>
       <mesh filename="file://$(find robotpadi_description)/meshes/arm_1.stl" scale="0.001 0.001 0.001"/>
@@ -218,5 +218,5 @@
   </visual>
   <collision>
-    <origin xyz="-2.741894 -0.284145 -0.962" rpy="0 0 0"/>
+    <origin xyz="-0.6435 -0.287 -0.962" rpy="0 0 0"/>
     <geometry>
       <mesh filename="file://$(find robotpadi_description)/meshes/arm_1.stl" scale="0.001 0.001 0.001"/>
@@ -225,5 +225,5 @@
 </link>
 <joint name="Revolute 1" type="continuous">
-  <origin xyz="2.868394 0.829145 0.965" rpy="0 0 0"/>
+  <origin xyz="0.77 0.832 0.965" rpy="0 0 0"/>
   <parent link="base_link"/>
   <child link="fr_steering_1"/>
@@ -231,5 +231,5 @@
 </joint>
 <joint name="Revolute 2" type="continuous">
-  <origin xyz="2.868394 -0.260855 0.965" rpy="0 0 0"/>
+  <origin xyz="0.77 -0.258 0.965" rpy="0 0 0"/>
   <parent link="base_link"/>
   <child link="br_steering_1"/>
@@ -237,5 +237,5 @@
 </joint>
 <joint name="Revolute 3" type="continuous">
-  <origin xyz="2.098394 0.829145 0.965" rpy="0 0 0"/>
+  <origin xyz="0.0 0.832 0.965" rpy="0 0 0"/>
   <parent link="base_link"/>
   <child link="fl_steering_1"/>
@@ -243,5 +243,5 @@
 </joint>
 <joint name="Revolute 4" type="continuous">
-  <origin xyz="2.098394 -0.260855 0.965" rpy="0 0 0"/>
+  <origin xyz="0.0 -0.258 0.965" rpy="0 0 0"/>
   <parent link="base_link"/>
   <child link="bl_steering_1"/>
@@ -252,5 +252,5 @@
   <parent link="br_steering_1"/>
   <child link="br_wheel_1"/>
-  <axis xyz="1.0 0.0 -0.0"/>
+  <axis xyz="1.0 -0.0 -0.0"/>
 </joint>
 <joint name="Revolute 6" type="continuous">
@@ -273,10 +273,10 @@
 </joint>
 <joint name="Rigid 9" type="fixed">
-  <origin xyz="4.581788 0.28129 1.027" rpy="0 0 0"/>
+  <origin xyz="0.385 0.287 1.027" rpy="0 0 0"/>
   <parent link="base_link"/>
   <child link="panel_1"/>
 </joint>
 <joint name="Rigid 10" type="fixed">
-  <origin xyz="2.741894 0.284145 0.962" rpy="0 0 0"/>
+  <origin xyz="0.6435 0.287 0.962" rpy="0 0 0"/>
   <parent link="base_link"/>
   <child link="arm_1"/>
