Commit message: update controller

File: install/robotpadi_description/share/robotpadi_description/urdf/materials.xacro (robot description, xacro)
@@ -1,15 +1 @@
-<?xml version="1.0" ?>
-<robot name="robotpadi" xmlns:xacro="http://www.ros.org/wiki/xacro" >
-<material name="silver">
-  <color rgba="0.700 0.700 0.700 1.000"/>
-</material>
-<material name="black">
-  <color rgba="0.000 0.000 0.000 1.000"/>
-</material>
-<material name="light_blue">
-  <color rgba="0.080 0.120 0.300 1.000"/>
-</material>
-<material name="yellow">
-  <color rgba="1.000 1.000 0.000 1.000"/>
-</material>
-</robot>
+/home/ubuntu/github/Omni-Directional-Mobile-Robot/build/robotpadi_description/urdf/materials.xacro

File: install/robotpadi_description/share/robotpadi_description/urdf/robotpadi.xacro (robot description, xacro)
@@ -1,284 +1 @@
-<?xml version="1.0" ?>
-<robot name="robotpadi" xmlns:xacro="http://www.ros.org/wiki/xacro">
-<xacro:include filename="$(find robotpadi_description)/urdf/materials.xacro" />
-<xacro:include filename="$(find robotpadi_description)/urdf/robotpadi.ros2control" />
-<xacro:include filename="$(find robotpadi_description)/urdf/robotpadi.gazebo" />
-<link name="base_link">
-  <inertial>
-    <origin xyz="0.38402832945911336 0.2840129113095087 1.0082275557140674" rpy="0 0 0"/>
-    <mass value="111.52248073403693"/>
-    <inertia ixx="19.278738" iyy="11.892444" izz="29.802061" ixy="0.058745" iyz="0.077376" ixz="0.004947"/>
-  </inertial>
-  <visual>
-    <origin xyz="0 0 0" rpy="0 0 0"/>
-    <geometry>
-      <mesh filename="file://$(find robotpadi_description)/meshes/base_link.stl" scale="0.001 0.001 0.001"/>
-    </geometry>
-    <material name="black"/>
-  </visual>
-  <collision>
-    <origin xyz="0 0 0" rpy="0 0 0"/>
-    <geometry>
-      <mesh filename="file://$(find robotpadi_description)/meshes/base_link.stl" scale="0.001 0.001 0.001"/>
-    </geometry>
-  </collision>
-</link>
-<link name="fr_steering_1">
-  <inertial>
-    <origin xyz="0.020209424438183965 -0.058184114298542866 -0.434806075320194" rpy="0 0 0"/>
-    <mass value="19.903337193485434"/>
-    <inertia ixx="0.720932" iyy="0.676639" izz="0.120784" ixy="0.017565" iyz="0.050773" ixz="-0.003917"/>
-  </inertial>
-  <visual>
-    <origin xyz="-0.77 -0.832 -0.965" rpy="0 0 0"/>
-    <geometry>
-      <mesh filename="file://$(find robotpadi_description)/meshes/fr_steering_1.stl" scale="0.001 0.001 0.001"/>
-    </geometry>
-    <material name="yellow"/>
-  </visual>
-  <collision>
-    <origin xyz="-0.77 -0.832 -0.965" rpy="0 0 0"/>
-    <geometry>
-      <mesh filename="file://$(find robotpadi_description)/meshes/fr_steering_1.stl" scale="0.001 0.001 0.001"/>
-    </geometry>
-  </collision>
-</link>
-<link name="br_steering_1">
-  <inertial>
-    <origin xyz="0.02067495895252003 0.05948919721980847 -0.42960566126027544" rpy="0 0 0"/>
-    <mass value="19.42819628224292"/>
-    <inertia ixx="0.69198" iyy="0.64895" izz="0.118365" ixy="-0.016967" iyz="-0.04479" ixz="-0.001759"/>
-  </inertial>
-  <visual>
-    <origin xyz="-0.77 0.258 -0.965" rpy="0 0 0"/>
-    <geometry>
-      <mesh filename="file://$(find robotpadi_description)/meshes/br_steering_1.stl" scale="0.001 0.001 0.001"/>
-    </geometry>
-    <material name="yellow"/>
-  </visual>
-  <collision>
-    <origin xyz="-0.77 0.258 -0.965" rpy="0 0 0"/>
-    <geometry>
-      <mesh filename="file://$(find robotpadi_description)/meshes/br_steering_1.stl" scale="0.001 0.001 0.001"/>
-    </geometry>
-  </collision>
-</link>
-<link name="fl_steering_1">
-  <inertial>
-    <origin xyz="-0.02067495895252023 -0.05948919721981982 -0.42960566126025335" rpy="0 0 0"/>
-    <mass value="19.42819628224292"/>
-    <inertia ixx="0.69198" iyy="0.64895" izz="0.118365" ixy="-0.016967" iyz="0.04479" ixz="0.001759"/>
-  </inertial>
-  <visual>
-    <origin xyz="0.0 -0.832 -0.965" rpy="0 0 0"/>
-    <geometry>
-      <mesh filename="file://$(find robotpadi_description)/meshes/fl_steering_1.stl" scale="0.001 0.001 0.001"/>
-    </geometry>
-    <material name="yellow"/>
-  </visual>
-  <collision>
-    <origin xyz="0.0 -0.832 -0.965" rpy="0 0 0"/>
-    <geometry>
-      <mesh filename="file://$(find robotpadi_description)/meshes/fl_steering_1.stl" scale="0.001 0.001 0.001"/>
-    </geometry>
-  </collision>
-</link>
-<link name="bl_steering_1">
-  <inertial>
-    <origin xyz="-0.02020942443818015 0.05818411429852913 -0.4348060753202161" rpy="0 0 0"/>
-    <mass value="19.903337193485434"/>
-    <inertia ixx="0.720932" iyy="0.676639" izz="0.120784" ixy="0.017565" iyz="-0.050773" ixz="0.003917"/>
-  </inertial>
-  <visual>
-    <origin xyz="0.0 0.258 -0.965" rpy="0 0 0"/>
-    <geometry>
-      <mesh filename="file://$(find robotpadi_description)/meshes/bl_steering_1.stl" scale="0.001 0.001 0.001"/>
-    </geometry>
-    <material name="yellow"/>
-  </visual>
-  <collision>
-    <origin xyz="0.0 0.258 -0.965" rpy="0 0 0"/>
-    <geometry>
-      <mesh filename="file://$(find robotpadi_description)/meshes/bl_steering_1.stl" scale="0.001 0.001 0.001"/>
-    </geometry>
-  </collision>
-</link>
-<link name="br_wheel_1">
-  <inertial>
-    <origin xyz="0.002000000000001445 8.992806499463768e-15 -8.326672684688674e-16" rpy="0 0 0"/>
-    <mass value="65.80472593736373"/>
-    <inertia ixx="1.584128" iyy="0.836383" izz="0.836383" ixy="0.0" iyz="0.0" ixz="0.0"/>
-  </inertial>
-  <visual>
-    <origin xyz="-0.858 0.258 -0.295" rpy="0 0 0"/>
-    <geometry>
-      <mesh filename="file://$(find robotpadi_description)/meshes/br_wheel_1.stl" scale="0.001 0.001 0.001"/>
-    </geometry>
-    <material name="black"/>
-  </visual>
-  <collision>
-    <origin xyz="-0.858 0.258 -0.295" rpy="0 0 0"/>
-    <geometry>
-      <mesh filename="file://$(find robotpadi_description)/meshes/br_wheel_1.stl" scale="0.001 0.001 0.001"/>
-    </geometry>
-  </collision>
-</link>
-<link name="fl_wheel_1">
-  <inertial>
-    <origin xyz="-0.0020000000000005708 -8.770761894538737e-15 2.398081733190338e-14" rpy="0 0 0"/>
-    <mass value="65.80472593736373"/>
-    <inertia ixx="1.584128" iyy="0.836383" izz="0.836383" ixy="0.0" iyz="0.0" ixz="0.0"/>
-  </inertial>
-  <visual>
-    <origin xyz="0.088 -0.832 -0.295" rpy="0 0 0"/>
-    <geometry>
-      <mesh filename="file://$(find robotpadi_description)/meshes/fl_wheel_1.stl" scale="0.001 0.001 0.001"/>
-    </geometry>
-    <material name="black"/>
-  </visual>
-  <collision>
-    <origin xyz="0.088 -0.832 -0.295" rpy="0 0 0"/>
-    <geometry>
-      <mesh filename="file://$(find robotpadi_description)/meshes/fl_wheel_1.stl" scale="0.001 0.001 0.001"/>
-    </geometry>
-  </collision>
-</link>
-<link name="bl_wheel_1">
-  <inertial>
-    <origin xyz="-0.002000000000001237 -8.493206138382448e-15 -6.661338147750939e-16" rpy="0 0 0"/>
-    <mass value="65.80472593736373"/>
-    <inertia ixx="1.584128" iyy="0.836383" izz="0.836383" ixy="0.0" iyz="0.0" ixz="0.0"/>
-  </inertial>
-  <visual>
-    <origin xyz="0.088 0.258 -0.295" rpy="0 0 0"/>
-    <geometry>
-      <mesh filename="file://$(find robotpadi_description)/meshes/bl_wheel_1.stl" scale="0.001 0.001 0.001"/>
-    </geometry>
-    <material name="black"/>
-  </visual>
-  <collision>
-    <origin xyz="0.088 0.258 -0.295" rpy="0 0 0"/>
-    <geometry>
-      <mesh filename="file://$(find robotpadi_description)/meshes/bl_wheel_1.stl" scale="0.001 0.001 0.001"/>
-    </geometry>
-  </collision>
-</link>
-<link name="fr_wheel_1">
-  <inertial>
-    <origin xyz="0.0019999999999994467 7.549516567451064e-15 2.4313884239290928e-14" rpy="0 0 0"/>
-    <mass value="65.80472593736373"/>
-    <inertia ixx="1.584128" iyy="0.836383" izz="0.836383" ixy="0.0" iyz="0.0" ixz="0.0"/>
-  </inertial>
-  <visual>
-    <origin xyz="-0.858 -0.832 -0.295" rpy="0 0 0"/>
-    <geometry>
-      <mesh filename="file://$(find robotpadi_description)/meshes/fr_wheel_1.stl" scale="0.001 0.001 0.001"/>
-    </geometry>
-    <material name="black"/>
-  </visual>
-  <collision>
-    <origin xyz="-0.858 -0.832 -0.295" rpy="0 0 0"/>
-    <geometry>
-      <mesh filename="file://$(find robotpadi_description)/meshes/fr_wheel_1.stl" scale="0.001 0.001 0.001"/>
-    </geometry>
-  </collision>
-</link>
-<link name="panel_1">
-  <inertial>
-    <origin xyz="4.287126209590042e-13 -5.242174278385914e-06 0.287647550111215" rpy="0 0 0"/>
-    <mass value="131.93512225471943"/>
-    <inertia ixx="26.841833" iyy="21.913769" izz="48.508633" ixy="0.0" iyz="-6.5e-05" ixz="0.0"/>
-  </inertial>
-  <visual>
-    <origin xyz="-0.385 -0.287 -1.027" rpy="0 0 0"/>
-    <geometry>
-      <mesh filename="file://$(find robotpadi_description)/meshes/panel_1.stl" scale="0.001 0.001 0.001"/>
-    </geometry>
-    <material name="light_blue"/>
-  </visual>
-  <collision>
-    <origin xyz="-0.385 -0.287 -1.027" rpy="0 0 0"/>
-    <geometry>
-      <mesh filename="file://$(find robotpadi_description)/meshes/panel_1.stl" scale="0.001 0.001 0.001"/>
-    </geometry>
-  </collision>
-</link>
-<link name="arm_1">
-  <inertial>
-    <origin xyz="-0.2584017212277529 0.0021110751355971624 -0.07218922154687024" rpy="0 0 0"/>
-    <mass value="22.7414514992095"/>
-    <inertia ixx="1.72933" iyy="1.730341" izz="3.147968" ixy="0.000336" iyz="0.000291" ixz="-0.001081"/>
-  </inertial>
-  <visual>
-    <origin xyz="-0.6435 -0.287 -0.962" rpy="0 0 0"/>
-    <geometry>
-      <mesh filename="file://$(find robotpadi_description)/meshes/arm_1.stl" scale="0.001 0.001 0.001"/>
-    </geometry>
-    <material name="silver"/>
-  </visual>
-  <collision>
-    <origin xyz="-0.6435 -0.287 -0.962" rpy="0 0 0"/>
-    <geometry>
-      <mesh filename="file://$(find robotpadi_description)/meshes/arm_1.stl" scale="0.001 0.001 0.001"/>
-    </geometry>
-  </collision>
-</link>
-<joint name="Revolute 1" type="continuous">
-  <origin xyz="0.77 0.832 0.965" rpy="0 0 0"/>
-  <parent link="base_link"/>
-  <child link="fr_steering_1"/>
-  <axis xyz="-0.0 0.0 -1.0"/>
-</joint>
-<joint name="Revolute 2" type="continuous">
-  <origin xyz="0.77 -0.258 0.965" rpy="0 0 0"/>
-  <parent link="base_link"/>
-  <child link="br_steering_1"/>
-  <axis xyz="-0.0 0.0 -1.0"/>
-</joint>
-<joint name="Revolute 3" type="continuous">
-  <origin xyz="0.0 0.832 0.965" rpy="0 0 0"/>
-  <parent link="base_link"/>
-  <child link="fl_steering_1"/>
-  <axis xyz="-0.0 0.0 -1.0"/>
-</joint>
-<joint name="Revolute 4" type="continuous">
-  <origin xyz="0.0 -0.258 0.965" rpy="0 0 0"/>
-  <parent link="base_link"/>
-  <child link="bl_steering_1"/>
-  <axis xyz="-0.0 0.0 -1.0"/>
-</joint>
-<joint name="Revolute 5" type="continuous">
-  <origin xyz="0.088 0.0 -0.67" rpy="0 0 0"/>
-  <parent link="br_steering_1"/>
-  <child link="br_wheel_1"/>
-  <axis xyz="1.0 -0.0 -0.0"/>
-</joint>
-<joint name="Revolute 6" type="continuous">
-  <origin xyz="-0.088 0.0 -0.67" rpy="0 0 0"/>
-  <parent link="fl_steering_1"/>
-  <child link="fl_wheel_1"/>
-  <axis xyz="-1.0 -0.0 0.0"/>
-</joint>
-<joint name="Revolute 7" type="continuous">
-  <origin xyz="-0.088 0.0 -0.67" rpy="0 0 0"/>
-  <parent link="bl_steering_1"/>
-  <child link="bl_wheel_1"/>
-  <axis xyz="-1.0 0.0 0.0"/>
-</joint>
-<joint name="Revolute 8" type="continuous">
-  <origin xyz="0.088 0.0 -0.67" rpy="0 0 0"/>
-  <parent link="fr_steering_1"/>
-  <child link="fr_wheel_1"/>
-  <axis xyz="1.0 0.0 -0.0"/>
-</joint>
-<joint name="Rigid 9" type="fixed">
-  <origin xyz="0.385 0.287 1.027" rpy="0 0 0"/>
-  <parent link="base_link"/>
-  <child link="panel_1"/>
-</joint>
-<joint name="Rigid 10" type="fixed">
-  <origin xyz="0.6435 0.287 0.962" rpy="0 0 0"/>
-  <parent link="base_link"/>
-  <child link="arm_1"/>
-</joint>
-</robot>
+/home/ubuntu/github/Omni-Directional-Mobile-Robot/build/robotpadi_description/urdf/robotpadi.xacro

File: src/robotpadi_description/urdf/robotpadi.xacro (robot description, xacro)
@@ -4,5 +4,11 @@
 <xacro:include filename="$(find robotpadi_description)/urdf/robotpadi.ros2control" />
 <xacro:include filename="$(find robotpadi_description)/urdf/robotpadi.gazebo" />
-<link name="base_link">
+<link name="base_link"/>
+<joint name="base_link_joint" type="fixed">
+  <parent link="base_link"/>
+  <child link="base_robot"/>
+  <origin xyz="0 0 0.92" rpy="0 0 0"/>  <!-- Raise base_link by the offset -->
+</joint>
+<link name="base_robot">
   <inertial>
     <origin xyz="4.7605171811971384e-05 7.503713021135889e-06 -1.28855617148301e-05" rpy="0 0 0"/>
@@ -15,5 +21,5 @@
       <mesh filename="file://$(find robotpadi_description)/meshes/base_link.stl" scale="0.001 0.001 0.001"/>
     </geometry>
-    <material name="silver"/>
+    <material name="black"/>
   </visual>
   <collision>
@@ -35,5 +41,5 @@
       <mesh filename="file://$(find robotpadi_description)/meshes/fr_steering_1.stl" scale="0.001 0.001 0.001"/>
     </geometry>
-    <material name="silver"/>
+    <material name="yellow"/>
   </visual>
   <collision>
@@ -55,5 +61,5 @@
       <mesh filename="file://$(find robotpadi_description)/meshes/br_steering_1.stl" scale="0.001 0.001 0.001"/>
     </geometry>
-    <material name="silver"/>
+    <material name="yellow"/>
   </visual>
   <collision>
@@ -75,5 +81,5 @@
       <mesh filename="file://$(find robotpadi_description)/meshes/fl_steering_1.stl" scale="0.001 0.001 0.001"/>
     </geometry>
-    <material name="silver"/>
+    <material name="yellow"/>
   </visual>
   <collision>
@@ -95,5 +101,5 @@
       <mesh filename="file://$(find robotpadi_description)/meshes/bl_steering_1.stl" scale="0.001 0.001 0.001"/>
     </geometry>
-    <material name="silver"/>
+    <material name="yellow"/>
   </visual>
   <collision>
@@ -115,5 +121,5 @@
       <mesh filename="file://$(find robotpadi_description)/meshes/br_wheel_1.stl" scale="0.001 0.001 0.001"/>
     </geometry>
-    <material name="silver"/>
+    <material name="black"/>
   </visual>
   <collision>
@@ -135,5 +141,5 @@
       <mesh filename="file://$(find robotpadi_description)/meshes/fl_wheel_1.stl" scale="0.001 0.001 0.001"/>
     </geometry>
-    <material name="silver"/>
+    <material name="black"/>
   </visual>
   <collision>
@@ -155,5 +161,5 @@
       <mesh filename="file://$(find robotpadi_description)/meshes/bl_wheel_1.stl" scale="0.001 0.001 0.001"/>
     </geometry>
-    <material name="silver"/>
+    <material name="black"/>
   </visual>
   <collision>
@@ -175,5 +181,5 @@
       <mesh filename="file://$(find robotpadi_description)/meshes/fr_wheel_1.stl" scale="0.001 0.001 0.001"/>
     </geometry>
-    <material name="silver"/>
+    <material name="black"/>
   </visual>
   <collision>
@@ -195,5 +201,5 @@
       <mesh filename="file://$(find robotpadi_description)/meshes/panel_1.stl" scale="0.001 0.001 0.001"/>
     </geometry>
-    <material name="silver"/>
+    <material name="light_blue"/>
   </visual>
   <collision>
@@ -226,5 +232,5 @@
 <joint name="Revolute 1" type="continuous">
   <origin xyz="0.386019 0.547995 -0.04324" rpy="0 0 0"/>
-  <parent link="base_link"/>
+  <parent link="base_robot"/>
   <child link="fr_steering_1"/>
   <axis xyz="-0.0 0.0 -1.0"/>
@@ -232,5 +238,5 @@
 <joint name="Revolute 2" type="continuous">
   <origin xyz="0.386019 -0.542005 -0.04324" rpy="0 0 0"/>
-  <parent link="base_link"/>
+  <parent link="base_robot"/>
   <child link="br_steering_1"/>
   <axis xyz="-0.0 0.0 -1.0"/>
@@ -238,5 +244,5 @@
 <joint name="Revolute 3" type="continuous">
   <origin xyz="-0.383981 0.547995 -0.04324" rpy="0 0 0"/>
-  <parent link="base_link"/>
+  <parent link="base_robot"/>
   <child link="fl_steering_1"/>
   <axis xyz="-0.0 0.0 -1.0"/>
@@ -244,5 +250,5 @@
 <joint name="Revolute 4" type="continuous">
   <origin xyz="-0.383981 -0.542005 -0.04324" rpy="0 0 0"/>
-  <parent link="base_link"/>
+  <parent link="base_robot"/>
   <child link="bl_steering_1"/>
   <axis xyz="-0.0 0.0 -1.0"/>
@@ -274,10 +280,10 @@
 <joint name="Rigid 9" type="fixed">
   <origin xyz="0.001019 0.002995 0.01876" rpy="0 0 0"/>
-  <parent link="base_link"/>
+  <parent link="base_robot"/>
   <child link="panel_1"/>
 </joint>
 <joint name="Rigid 10" type="fixed">
   <origin xyz="0.259519 0.002995 -0.04624" rpy="0 0 0"/>
-  <parent link="base_link"/>
+  <parent link="base_robot"/>
   <child link="arm_1"/>
 </joint>
